File: PCB/Jasmine v1.kicad_sch (KiCad schematic)
At the start: 153 parts, among them J2 ARGB, SW1 SW_PUSH_LED, SW2 SW_PUSH_LED, SW3 SW_PUSH_LED, U3 RP2040_Pro_Micro

Commit message: fixed schem
Parts:
- removed D18, D51, D52: 1N4148W, ScottoKeebs_Components:Diode_SOD-123, symbol Diode:1N4148W
- removed SW1, SW2, SW3: SW_PUSH_LED, ScottoKeebs_Components:LED_SK6812MINI, symbol SofleKeyboard:SW_PUSH_LED
Connections:
- net col10: no longer MX66.1
- net col15: now also MX51.1
- net col16: no longer MX51.1
- net col9: now also MX66.1
- net row3: no longer MX66.2
- net at MX18.2: now also D17.2 (A), MX17.2
- net at D49.2 (A), MX49.2: now also MX51.2
- net at D50.2 (A), MX50.2: now also MX52.2
- net at D58.2 (A), MX58.2: now also MX66.2
Other:
- moved on the sheet: MX18, MX51, MX52, MX66
